File: hardware/0.1/rf-sig-gen.kicad_pcb (KiCad board)
At the start: 4 copper layers, 50 x 22.9 mm, 91 parts, among them J1 Feather, J2 SMA, U1 MAX2871, U2 LP5912, U3 MIC5366-1.8, U4 SKY12347-362LF, U5 TRF37A75, U6 AD8319, U7 STP08CP05

Commit message: final changes
Routing:
- net GND: track 83.2 -> 86.1 mm, vias 122 -> 121
Other:
- board text added: "JLCJLC JLCJLC"
